File: ProjectDrive.kicad_pcb (KiCad board)
At the start: 2 copper layers, 131.5 x 74.6 mm, 33 parts, among them U1 RP2040_Zero

Commit message: Updated PCB
Parts:
- removed D1, D10, D11, D12, D13, D14, D15, D16, D2, D3, D4, D5, D6, D7, D8, D9: Diode, ScottoKeebs_Components:Diode_DO-35
- added REF**: MountingHole_2.2mm_M2, MountingHole:MountingHole_2.2mm_M2, F.Cu at (112.9, 116.4)
- added REF**: MountingHole_2.2mm_M2, MountingHole:MountingHole_2.2mm_M2, F.Cu at (113.2, 50.8)
- added REF**: MountingHole_2.2mm_M2, MountingHole:MountingHole_2.2mm_M2, F.Cu at (235.4, 116.5)
- added REF**: MountingHole_2.2mm_M2, MountingHole:MountingHole_2.2mm_M2, F.Cu at (235.7, 50.9)
Connections:
- S1 pad 1: unconnected-(S1-Pad1) -> Up
- S1 pad 2: Net-(D1-A) -> GND
- S10 pad 1: unconnected-(S10-Pad1) -> 3K
- S10 pad 2: Net-(D10-A) -> GND
- S11 pad 1: unconnected-(S11-Pad1) -> Start
- S11 pad 2: Net-(D11-A) -> GND
- S12 pad 1: unconnected-(S12-Pad1) -> Select
- S12 pad 2: Net-(D12-A) -> GND
- S13 pad 1: unconnected-(S13-Pad1) -> Home
- S13 pad 2: Net-(D13-A) -> GND
- S14 pad 1: unconnected-(S14-Pad1) -> 4K
- S14 pad 2: Net-(D14-A) -> GND
- S15 pad 1: unconnected-(S15-Pad1) -> 4P
- S15 pad 2: Net-(D15-A) -> GND
- S16 pad 1: unconnected-(S16-Pad1) -> Touchpad
- S16 pad 2: Net-(D16-A) -> GND
- S2 pad 1: unconnected-(S2-Pad1) -> Down
- S2 pad 2: Net-(D2-A) -> GND
- S3 pad 1: unconnected-(S3-Pad1) -> Left
- S3 pad 2: Net-(D3-A) -> GND
- S4 pad 1: unconnected-(S4-Pad1) -> Right
- S4 pad 2: Net-(D4-A) -> GND
- S5 pad 1: unconnected-(S5-Pad1) -> 1P
- S5 pad 2: Net-(D5-A) -> GND
- S6 pad 1: unconnected-(S6-Pad1) -> 2P
- S6 pad 2: Net-(D6-A) -> GND
- S7 pad 1: unconnected-(S7-Pad1) -> 3P
- S7 pad 2: Net-(D7-A) -> GND
- S8 pad 1: unconnected-(S8-Pad1) -> 1K
- S8 pad 2: Net-(D8-A) -> GND
- S9 pad 1: unconnected-(S9-Pad1) -> 2K
- S9 pad 2: Net-(D9-A) -> GND
Routing:
- net 3K: track 106.6 -> 70.8 mm, vias 0 -> 2
- net Net-(D14-A): track 15.8 -> 0.00 mm
- net 3P: track 45.1 -> 60.3 mm
- net 2P: track 38.3 -> 52.5 mm
- net Select: track 45.8 -> 58.4 mm, vias 0 -> 2
- net Net-(D15-A): track 12.4 -> 0.00 mm
- net Net-(D2-A): track 11.9 -> 0.00 mm
- net Down: track 49.8 -> 61.4 mm
- net 1P: track 32.6 -> 43.9 mm
- net Net-(D3-A): track 11.0 -> 0.00 mm
- net Net-(D4-A): track 10.8 -> 0.00 mm
- net Net-(D8-A): track 10.6 -> 0.00 mm
- net Net-(D1-A): track 10.6 -> 0.00 mm
- net Net-(D5-A): track 10.5 -> 0.00 mm
- net Net-(D11-A): track 10.4 -> 0.00 mm
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