File: ProjectDrive.kicad_sch (KiCad schematic)
At the start: 33 parts, among them U1 RP2040_Zero

Commit message: Updated PCB
Parts:
- removed D1, D10, D11, D12, D13, D14, D15, D16, D2, D3, D4, D5, D6, D7, D8, D9: Diode, ScottoKeebs_Components:Diode_DO-35, symbol ScottoKeebs:Placeholder_Diode
Connections:
- net 1K: now also S8.1
- net 1P: now also S5.1
- net 2K: now also S9.1
- net 2P: now also S6.1
- net 3K: now also S10.1
- net 3P: now also S7.1
- net 4K: now also S14.1
- net 4P: now also S15.1
- net Down: now also S2.1
- net GND: now also S1.2, S10.2, S11.2, S12.2, S13.2, S14.2, S15.2, S16.2, S2.2, S3.2, S4.2, S5.2, S6.2, S7.2, S8.2, S9.2
- net Home: now also S13.1
- net Left: now also S3.1
- net Right: now also S4.1
- net Select: now also S12.1
- net Start: now also S11.1
- net Touchpad: now also S16.1
- net Up: now also S1.1
